File: hardware/kicad/maidenhead-pocket-locator.sch (KiCad schematic (older format))
At the start: 13 parts, among them J1 USB-C: VBUS,CC1,CC2,D+,D-,GND, J2 BAT+,NTC,GND, J3 LCD: GND,5V,VO,RS,RW,E,D0-D7,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, Q1 DMP3098L signal PMOS, Q2 DMN2050L hold NMOS, U1 RP2040 QFN56 — see pin map, U2 W25Q16: CS,DO,WP,GND,DI,CLK,H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, U3 BQ24074: IN,BAT,TS,EN2,EN1,TM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, U4 TPS63802: VIN,L1,L2,VOUT,FB,E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, U5 TPS61023: FB,EN,VIN,GND,SW,VO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, U6 SN74LVC8T245: VCCA/A0-A5/DIR/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, U7 GP-02: VCC,GND,TX,RX,PPS,RF, U8 TPS22916 GNSS load switch

Commit message: Finish pocket locator project sources
Parts:
- removed J1: USB-C: VBUS,CC1,CC2,D+,D-,GND, symbol Connector_Generic:Conn_01x06
- removed J2: BAT+,NTC,GND, symbol Connector_Generic:Conn_01x03
- removed J3: LCD: GND,5V,VO,RS,RW,E,D0-D7,BL+,BL-, symbol Connector_Generic:Conn_01x16
- removed Q1: DMP3098L signal PMOS, symbol Connector_Generic:Conn_01x03
- removed Q2: DMN2050L hold NMOS, symbol Connector_Generic:Conn_01x03
- removed U1: RP2040 QFN56 — see pin map, symbol Connector_Generic:Conn_02x20_Odd_Even
- removed U2: W25Q16: CS,DO,WP,GND,DI,CLK,HOLD,VCC, symbol Connector_Generic:Conn_01x08
- removed U3: BQ24074: IN,BAT,TS,EN2,EN1,TMR,CE,CHG,OUT,ILIM,IS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, symbol Connector_Generic:Conn_01x14
- removed U4: TPS63802: VIN,L1,L2,VOUT,FB,EN,MODE,PG,GND, symbol Connector_Generic:Conn_01x09
- removed U5: TPS61023: FB,EN,VIN,GND,SW,VOUT, symbol Connector_Generic:Conn_01x06
- removed U6: SN74LVC8T245: VCCA/A0-A5/DIR/OE/B0-B5/VCCB/GND, symbol Connector_Generic:Conn_02x12_Odd_Even
- removed U7: GP-02: VCC,GND,TX,RX,PPS,RF, symbol Connector_Generic:Conn_01x06
- removed U8: TPS22916 GNSS load switch, symbol Connector_Generic:Conn_01x06
- added C1: 100nF, Capacitor_SMD:C_0402_1005Metric, symbol PL_C1
- added C2: 100nF, Capacitor_SMD:C_0402_1005Metric, symbol PL_C2
- added C3: 100nF, Capacitor_SMD:C_0402_1005Metric, symbol PL_C3
- added C4: 100nF, Capacitor_SMD:C_0402_1005Metric, symbol PL_C4
- added C5: 100nF, Capacitor_SMD:C_0402_1005Metric, symbol PL_C5
- added C6: 100nF, Capacitor_SMD:C_0402_1005Metric, symbol PL_C6
- added C7: 100nF, Capacitor_SMD:C_0402_1005Metric, symbol PL_C7
- added C8: 100nF, Capacitor_SMD:C_0402_1005Metric, symbol PL_C8
- added C9: 100nF, Capacitor_SMD:C_0402_1005Metric, symbol PL_C9
- added CADC1: 1uF, Capacitor_SMD:C_0603_1608Metric, symbol PL_CADC1
- added CBAT1: 4.7uF, Capacitor_SMD:C_0603_1608Metric, symbol PL_CBAT1
- added CBATADC1: 100nF, Capacitor_SMD:C_0402_1005Metric, symbol PL_CBATADC1
- added CBBIN1: 10uF, Capacitor_SMD:C_0805_2012Metric, symbol PL_CBBIN1
- added CBBOUT1: 22uF, Capacitor_SMD:C_0805_2012Metric, symbol PL_CBBOUT1
- added CDV1: 100nF, Capacitor_SMD:C_0402_1005Metric, symbol PL_CDV1
- added CDV2: 100nF, Capacitor_SMD:C_0402_1005Metric, symbol PL_CDV2
- added CFLASH1: 100nF, Capacitor_SMD:C_0402_1005Metric, symbol PL_CFLASH1
- added CGIN1: 1uF, Capacitor_SMD:C_0402_1005Metric, symbol PL_CGIN1
- added CGNSS1: 100nF, Capacitor_SMD:C_0402_1005Metric, symbol PL_CGNSS1
- added CGNSS2: 820pF, Capacitor_SMD:C_0402_1005Metric, symbol PL_CGNSS2
- added CGNSS3: 10uF, Capacitor_SMD:C_0805_2012Metric, symbol PL_CGNSS3
- added CGOUT1: 4.7uF, Capacitor_SMD:C_0603_1608Metric, symbol PL_CGOUT1
- added CIN1: 1uF, Capacitor_SMD:C_0603_1608Metric, symbol PL_CIN1
- added CLCDIN1: 10uF, Capacitor_SMD:C_0805_2012Metric, symbol PL_CLCDIN1
- added CLCDO1: 10uF, Capacitor_SMD:C_0805_2012Metric, symbol PL_CLCDO1
- added CLCDO2: 10uF, Capacitor_SMD:C_0805_2012Metric, symbol PL_CLCDO2
- added COUT1: 4.7uF, Capacitor_SMD:C_0603_1608Metric, symbol PL_COUT1
- added CRESET1: 100nF, Capacitor_SMD:C_0402_1005Metric, symbol PL_CRESET1
- added CULD1: 100nF, Capacitor_SMD:C_0402_1005Metric, symbol PL_CULD1
- added CULS1: 100nF, Capacitor_SMD:C_0402_1005Metric, symbol PL_CULS1
- added CVREG1: 1uF, Capacitor_SMD:C_0603_1608Metric, symbol PL_CVREG1
- added CX1: 15pF, Capacitor_SMD:C_0402_1005Metric, symbol PL_CX1
- added CX2: 15pF, Capacitor_SMD:C_0402_1005Metric, symbol PL_CX2
- added D1: TPD2EUSB30DRTR, PocketLocator:Texas_DRT0003A, symbol PL_D1
- added D2: BAT54H, Diode_SMD:D_SOD-323, symbol PL_D2
- added D3: 1N4148WS, Diode_SMD:D_SOD-323, symbol PL_D3
- added D4: BAT54H, Diode_SMD:D_SOD-323, symbol PL_D4
- added D5: 1N4148WS, Diode_SMD:D_SOD-323, symbol PL_D5
- added F1: MF-MSMF050-2, Fuse:Fuse_1812_4532Metric, symbol PL_F1
- added J1: USB4105-GF-A, PocketLocator:USB4105-GF-A, symbol PL_J1
- added J2: B3B-PH-K-S(LF)(SN), Connector_JST:JST_PH_B3B-PH-K_1x03_P2.00mm_Vertical, symbol PL_J2
- added J3: 61301611121, Connector_PinHeader_2.54mm:PinHeader_1x16_P2.54mm_Vertical, symbol PL_J3
- added J4: Hirose 20449-001E, Connector_Coaxial:U.FL_Hirose_U.FL-R-SMT-1_Vertical, symbol PL_J4
- added LBB1: XFL4020-471MEC, Inductor_SMD:L_Coilcraft_XxL4020, symbol PL_LBB1
- added LED1: KP-2012EC, LED_SMD:LED_0805_2012Metric, symbol PL_LED1
- added LLCD1: LQH2MCN1R0M02L, Inductor_SMD:L_0805_2012Metric, symbol PL_LLCD1
- added Q1: DMP3098L-7, Package_TO_SOT_SMD:SOT-23, symbol PL_Q1
- added Q2: DMN2050L-7, Package_TO_SOT_SMD:SOT-23, symbol PL_Q2
- added Q3: DMN2050L-7, Package_TO_SOT_SMD:SOT-23, symbol PL_Q3
- added Q4: DMP3098L-7, Package_TO_SOT_SMD:SOT-23, symbol PL_Q4
- added Q5: DMN2050L-7, Package_TO_SOT_SMD:SOT-23, symbol PL_Q5
- added RBAT1: 100k, Resistor_SMD:R_0402_1005Metric, symbol PL_RBAT1
- added RBAT2: 100k, Resistor_SMD:R_0402_1005Metric, symbol PL_RBAT2
- added RBATG1: 100k, Resistor_SMD:R_0402_1005Metric, symbol PL_RBATG1
- added RBB1: 511k, Resistor_SMD:R_0402_1005Metric, symbol PL_RBB1
- added RBB2: 91k, Resistor_SMD:R_0402_1005Metric, symbol PL_RBB2
- added RBL1: 68R, Resistor_SMD:R_0603_1608Metric, symbol PL_RBL1
- added RBOOT1: 1k, Resistor_SMD:R_0402_1005Metric, symbol PL_RBOOT1
- added RCC1: 5.1k, Resistor_SMD:R_0402_1005Metric, symbol PL_RCC1
- added RCC2: 5.1k, Resistor_SMD:R_0402_1005Metric, symbol PL_RCC2
- added RCHG1: 1k, Resistor_SMD:R_0402_1005Metric, symbol PL_RCHG1
- added RCHGPU1: 100k, Resistor_SMD:R_0402_1005Metric, symbol PL_RCHGPU1
- added REN1: 1M, Resistor_SMD:R_0402_1005Metric, symbol PL_REN1
- added RGNSSEN1: 100k, Resistor_SMD:R_0402_1005Metric, symbol PL_RGNSSEN1
- added RGNSSRX1: 33R, Resistor_SMD:R_0402_1005Metric, symbol PL_RGNSSRX1
- added RGNSSTX1: 33R, Resistor_SMD:R_0402_1005Metric, symbol PL_RGNSSTX1
- added RHOLD1: 100k, Resistor_SMD:R_0402_1005Metric, symbol PL_RHOLD1
- added RILIM1: 2.00k, Resistor_SMD:R_0402_1005Metric, symbol PL_RILIM1
- added RISET1: 2.20k, Resistor_SMD:R_0402_1005Metric, symbol PL_RISET1
- added RITERM1: 3.30k, Resistor_SMD:R_0402_1005Metric, symbol PL_RITERM1
- added RLCD1: 909k, Resistor_SMD:R_0402_1005Metric, symbol PL_RLCD1
- added RLCD2: 100k, Resistor_SMD:R_0402_1005Metric, symbol PL_RLCD2
- added RLCDEN1: 100k, Resistor_SMD:R_0402_1005Metric, symbol PL_RLCDEN1
- added RLOC1: 100k, Resistor_SMD:R_0402_1005Metric, symbol PL_RLOC1
- added ROFF1: 100k, Resistor_SMD:R_0402_1005Metric, symbol PL_ROFF1
- added RRESET1: 100k, Resistor_SMD:R_0402_1005Metric, symbol PL_RRESET1
- added RSENSEEN1: 100k, Resistor_SMD:R_0402_1005Metric, symbol PL_RSENSEEN1
- added RSTART1: 100k, Resistor_SMD:R_0402_1005Metric, symbol PL_RSTART1
- added RTMR1: 48.7k, Resistor_SMD:R_0402_1005Metric, symbol PL_RTMR1
- added RUSB1: 27R, Resistor_SMD:R_0402_1005Metric, symbol PL_RUSB1
- added RUSB2: 27R, Resistor_SMD:R_0402_1005Metric, symbol PL_RUSB2
- added RVB1: 82k, Resistor_SMD:R_0402_1005Metric, symbol PL_RVB1
- added RVB2: 100k, Resistor_SMD:R_0402_1005Metric, symbol PL_RVB2
- added RVO1: 4.7k, Resistor_SMD:R_0402_1005Metric, symbol PL_RVO1
- added RVO2: 560R, Resistor_SMD:R_0402_1005Metric, symbol PL_RVO2
- added RXTAL1: 1k, Resistor_SMD:R_0402_1005Metric, symbol PL_RXTAL1
- added SW1: TL1014BF160QG, PocketLocator:SW_TL1014B, symbol PL_SW1
- added SW2: TL1014BF160QG, PocketLocator:SW_TL1014B, symbol PL_SW2
- added SW3: EVQ-P7A01P, Button_Switch_SMD:SW_SPST_EVQP7A, symbol PL_SW3
- added SW4: EVQ-P7A01P, Button_Switch_SMD:SW_SPST_EVQP7A, symbol PL_SW4
- added TH1: 10k NTC DNP, Resistor_SMD:R_0603_1608Metric, symbol PL_TH1
- added TP1: VBUS, TestPoint:TestPoint_Pad_D1.5mm, symbol PL_TP1
- added TP10: SWDIO, TestPoint:TestPoint_Pad_D1.5mm, symbol PL_TP10
- added TP11: SWCLK, TestPoint:TestPoint_Pad_D1.5mm, symbol PL_TP11
- added TP12: RUN_N, TestPoint:TestPoint_Pad_D1.5mm, symbol PL_TP12
- added TP13: BOOTSEL_N, TestPoint:TestPoint_Pad_D1.5mm, symbol PL_TP13
- added TP2: BAT, TestPoint:TestPoint_Pad_D1.5mm, symbol PL_TP2
- added TP3: SYS_RAW, TestPoint:TestPoint_Pad_D1.5mm, symbol PL_TP3
- added TP4: 3V3, TestPoint:TestPoint_Pad_D1.5mm, symbol PL_TP4
- added TP5: 5V_LCD, TestPoint:TestPoint_Pad_D1.5mm, symbol PL_TP5
- added TP6: GND, TestPoint:TestPoint_Pad_D1.5mm, symbol PL_TP6
- added TP7: POWER_HOLD, TestPoint:TestPoint_Pad_D1.5mm, symbol PL_TP7
- added TP8: GNSS_TX, TestPoint:TestPoint_Pad_D1.5mm, symbol PL_TP8
- added TP9: GNSS_RX, TestPoint:TestPoint_Pad_D1.5mm, symbol PL_TP9
- added U1: RP2040, Package_DFN_QFN:QFN-56-1EP_7x7mm_P0.4mm_EP3.2x3.2mm, symbol PL_U1
- added U2: W25Q16JVUXIQ, PocketLocator:Winbond_UX_8, symbol PL_U2
- added U3: BQ24074RGTR, PocketLocator:Texas_RGT0016C, symbol PL_U3
- added U4: TPS63802DLAR, PocketLocator:Texas_DLA0010A, symbol PL_U4
- added U5: TPS61023DRLR, Package_TO_SOT_SMD:SOT-563, symbol PL_U5
- added U6: SN74LVC8T245PWR, Package_SO:TSSOP-24_4.4x7.8mm_P0.65mm, symbol PL_U6
- added U7: Ai-Thinker GP-02, PocketLocator:GP-02, symbol PL_U7
- added U8: TPS22916BYFPR, PocketLocator:Texas_YFP0004, symbol PL_U8
- added X1: ABM8-272-T3, Crystal:Crystal_SMD_Abracon_ABM8G-4Pin_3.2x2.5mm, symbol PL_X1
Connections:
- net labels added: BAT_SENSE_GATE, BAT_SENSE_SW, BOOTSEL_N, CHG_LED_A, GNSS_RX_U7, GNSS_TX_U7, LOCATE_RAW, VBUS_RAW, XOUT_XTAL
- wire segments 114 -> 355
- no-connect marks 0 -> 29
Other:
- note added: "BQ24074 OUT is the sole SYS_RAW source. J1 VBUS_RAW passes through F1 to VBUS."
- note added: "EXACT PAD-NUMBER NETLIST — all unassigned physical pads are explicit no-connects"
- note removed: "All reference passives, exact pin numbers, values, footprints and test points are captured in design.yaml, BOM and PCB."
- note removed: "GNSS / LCD"
- note removed: "POWER FLOW: USB-C VBUS -> BQ24074 IN; cell -> BAT; BQ24074 OUT -> SYS_RAW only."
- note removed: "RP2040 / FLASH / USB"
- note removed: "TPS63802 ENABLE LATCH / 3V3"
- note removed: "USB-C / BQ24074 POWER PATH"
